File: ShadowRunner.kicad_pcb (KiCad board)
At the start: 2 copper layers, 81 parts, among them J1 micro JST SH, J2 GRPB052VWQS-RC, J3 SIM_Card, J4 MM8130-2600, J5 U.FL-R-SMT-1, Q1 DMN65D8L, Q2 DMN65D8L, U1 LM1117-ADJ, U11 P822601, U2 USB-C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

Commit message: Layout improved.
Let's see if I'll be able to route this thing....
Parts:
- removed H1, H2, H3: MountingHole, MountingHole:MountingHole_2.5mm
- removed R41, R42, R43, R44, R45, R46, R47, R48, R49: 0, Resistor_SMD:R_01005_0402Metric
- removed U11: P822601, MyLibs:P822601
- added AE2: Antenna_Chip, MyLibs:PCS.06.A, F.Cu at (126.2, 101.5)
- C1, C11, C2, C3, C4, R1, R2, R3, R4, R7, R8, U1, U3, U6: moved to F.Cu
- J3: moved to B.Cu
- moved R2 127.0 mm to (117.0, 130.2), turned to 270 degrees
- moved R1 125.2 mm to (118.2, 130.2), turned to 270 degrees
- moved R4 124.9 mm to (108.9, 130.5), turned to 270 degrees
- moved R11 124.2 mm to (119.0, 118.2)
- moved C3 123.4 mm to (119.5, 130.2), turned to 270 degrees
- moved R3 123.1 mm to (110.1, 130.5), turned to 270 degrees
- moved R7 121.6 mm to (120.8, 130.2), turned to 90 degrees
- moved C4 121.3 mm to (111.4, 130.5), turned to 270 degrees
- moved C1 119.8 mm to (122.0, 130.2), turned to 270 degrees
- moved R8 119.6 mm to (112.7, 130.5), turned to 90 degrees
- moved U9 119.4 mm to (122.0, 116.8), turned to 180 degrees
- moved C2 117.8 mm to (113.9, 130.5), turned to 270 degrees
- moved U1 115.3 mm to (119.8, 124.7), turned to 90 degrees
- moved R12 114.8 mm to (141.2, 127.1)
- moved R15 114.8 mm to (140.0, 127.1)
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Connections:
- C10 pad 1: +1V8 -> Net-(C10-Pad1)
- C9 pad 1: +1V8 -> Net-(C10-Pad1)

Commit message: lots of routing
Parts:
- moved L1 6.25 mm to (124.8, 114.2)
- moved C8 4.70 mm to (124.8, 115.5), turned to 0 degrees
- moved C20 4.04 mm to (152.7, 111.5), turned to 0 degrees
- moved C22 2.79 mm to (154.0, 117.7)
- moved C21 2.56 mm to (152.8, 124.0), turned to 0 degrees
- moved D5 2.51 mm to (107.5, 128.0)
- moved C1 0.25 mm to (122.0, 130.5)
- moved C3 0.25 mm to (119.5, 130.5)
- moved R1 0.25 mm to (118.2, 130.5)
- moved R2 0.25 mm to (117.0, 130.5)
- moved R22 0.25 mm to (104.2, 118.2)
- moved R7 0.25 mm to (120.8, 130.5)
- moved U1 0.25 mm to (119.8, 124.9)
- moved U8 0.25 mm to (110.0, 116.8)
- turned D1 to 180 degrees
Routing:
- net +1V8: track 0.00 -> 93.3 mm, vias 0 -> 6
- net +3V3: track 0.00 -> 89.5 mm, vias 0 -> 2
- net GND: track 0.00 -> 63.0 mm, vias 0 -> 6
- net Net-(R22-Pad2): track 0.00 -> 55.0 mm
- net Net-(R11-Pad2): track 0.00 -> 40.9 mm
- net VBUS: track 0.00 -> 37.7 mm, vias 0 -> 1
- net SWRESET: track 0.00 -> 32.8 mm, vias 0 -> 2
- net SWDCLK: track 0.00 -> 32.6 mm, vias 0 -> 2
- net SWDIO: track 0.00 -> 28.2 mm, vias 0 -> 2
- net Net-(R16-Pad2): track 0.00 -> 15.8 mm, vias 0 -> 2
- net Net-(D2-Pad1): track 0.00 -> 15.0 mm, vias 0 -> 2
- net Net-(R6-Pad1): track 0.00 -> 13.1 mm, vias 0 -> 1
- net Net-(R1-Pad2): track 0.00 -> 12.6 mm, vias 0 -> 2
- net Net-(R3-Pad2): track 0.00 -> 11.3 mm, vias 0 -> 2
- net Net-(R15-Pad2): track 0.00 -> 10.8 mm
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