File: ShadowRunner.sch (KiCad schematic (older format))
At the start: 69 parts, among them J1 micro JST SH, J2 GRPB052VWQS-RC, J3 SIM_Card, J4 MM8130-2600, J5 U.FL-R-SMT-1, Q1 DMN65D8L, Q2 DMN65D8L, U1 LM1117-ADJ, U2 USB-C, U3 LM1117-ADJ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

Commit message: All connections made
Parts:
- removed AE2: Antenna_Chip, MyLibs:PCS.06.A, symbol Device:Antenna_Chip
- added J6: PCS.06.A, MyLibs:PCS.06.A, symbol myPartsLibrary:PCS.06.A
- D5: value DIODE -> PMEG2020EPK,315; footprint Diode_SMD:D_0402_1005Metric -> MyLibs:D_0603_1608Metric_Pad1.05x0.95mm_HandSolder
Connections:
- net +1V8: now also C16.2, L5.2
- net +3V3: no longer C16.2, L5.2
- net GND: now also J6.1 (Pin_1), J6.2 (Pin_2), J6.3 (Pin_3)
- net at C12.1, L3.1: now also J6.4 (Pin_4)
- no-connect marks 79 -> 80
Other:
- note added: "1A"
Changed lines of the file:
@@
-$EndComp
-$Comp
-L power:+3V3 #PWR047
-U 1 1 5E86AF56
-P 11450 2500
-F 0 "#PWR047" H 11450 2350 50  0001 C CNN
-F 1 "+3V3" H 11465 2673 50  0000 C CNN
-F 2 "" H 11450 2500 50  0001 C CNN
-F 3 "" H 11450 2500 50  0001 C CNN
-	1    11450 2500
-	1    0    0    -1
 $EndComp
 $Comp
@@
 	1    0    0    -1
 $EndComp
-Text Notes 800  3450 0    50   ~ 0
-ASR00012
-$Comp
-L power:GND #PWR011
-U 1 1 5F578384
-P 1400 3350
-F 0 "#PWR011" H 1400 3100 50  0001 C CNN
-F 1 "GND" H 1405 3177 50  0000 C CNN
-F 2 "" H 1400 3350 50  0001 C CNN
-F 3 "" H 1400 3350 50  0001 C CNN
-	1    1400 3350
-	1    0    0    -1
-$EndComp
-$Comp
-L power:VBUS #PWR010
-U 1 1 5F5B0AAB
-P 1400 3000
-F 0 "#PWR010" H 1400 2850 50  0001 C CNN
-F 1 "VBUS" H 1415 3173 50  0000 C CNN
-F 2 "" H 1400 3000 50  0001 C CNN
-F 3 "" H 1400 3000 50  0001 C CNN
-	1    1400 3000
-	1    0    0    -1
-$EndComp
-Wire Wire Line
-	1150 3150 1400 3150
-Wire Wire Line
-	1400 3150 1400 3000
-Wire Wire Line
-	1400 3350 1400 3250
-Wire Wire Line
-	1150 3250 1400 3250
 Text Notes 2950 2900 0    50   ~ 0
 VERIFY FOOTPRINT!!
@@
 	1800 9700 1800 10000
 NoConn ~ 1700 9900
-$Comp
-L Connector_Generic:Conn_01x02 J1
-U 1 1 5F4B3C2C
-P 950 3150
-F 0 "J1" H 868 3367 50  0000 C CNN
-F 1 " micro JST SH" H 868 3276 50  0000 C CNN
-F 2 "MyLibs:S2B-ZR-SM4A-TFLFSN" H 950 3150 50  0001 C CNN
-F 3 "~" H 950 3150 50  0001 C CNN
-	1    950  3150
-	-1   0    0    -1
-$EndComp
 Text Notes 700  2700 0    50   ~ 0
 S2B-ZR-SM4A-TF(LF)(SN)
@@
 P 2850 850
 F 0 "D5" H 2700 800 50  0000 C CNN
-F 1 "DIODE" H 3050 750 50  0000 C CNN
-F 2 "Diode_SMD:D_0402_1005Metric" H 2850 850 50  0001 C CNN
+F 1 "PMEG2020EPK,315" H 2600 1000 50  0000 C CNN
+F 2 "MyLibs:D_0603_1608Metric_Pad1.05x0.95mm_HandSolder" H 2850 850 50  0001 C CNN
 F 3 "~" H 2850 850 50  0001 C CNN
 	1    2850 850
@@
 Wire Wire Line
 	10950 7900 14300 7900
-$Comp
-L Device:Antenna_Chip AE2
-U 1 1 607D025F
-P 9300 1200
-F 0 "AE2" H 9156 1327 50  0000 R CNN
-F 1 "Antenna_Chip" H 9156 1236 50  0000 R CNN
-F 2 "MyLibs:PCS.06.A" H 9200 1375 50  0001 C CNN
-F 3 "~" H 9200 1375 50  0001 C CNN
-	1    9300 1200
-	-1   0    0    -1
-$EndComp
-$Comp
-L power:GND #PWR0106
-U 1 1 6083E10A
-P 9200 1350
-F 0 "#PWR0106" H 9200 1100 50  0001 C CNN
-F 1 "GND" H 9100 1200 50  0000 C CNN
-F 2 "" H 9200 1350 50  0001 C CNN
-F 3 "" H 9200 1350 50  0001 C CNN
-	1    9200 1350
-	1    0    0    -1
-$EndComp
-Wire Wire Line
-	9200 1300 9200 1350
 Wire Wire Line
 	9400 1300 9650 1300
 Connection ~ 9650 1300
 $Comp
-L power:+1V8 #PWR?
+L power:+1V8 #PWR0106
 U 1 1 60C9BA0A
 P 8250 2500
-F 0 "#PWR?" H 8250 2350 50  0001 C CNN
+F 0 "#PWR0106" H 8250 2350 50  0001 C CNN
 F 1 "+1V8" H 8265 2673 50  0000 C CNN
 F 2 "" H 8250 2500 50  0001 C CNN
@@
 	1    0    0    -1
 $EndComp
+NoConn ~ 5550 1200
+$Comp
+L myPartsLibrary:PCS.06.A J6
+U 1 1 60FA87E2
+P 9150 1150
+F 0 "J6" H 9167 1515 50  0000 C CNN
+F 1 "PCS.06.A" H 9167 1424 50  0000 C CNN
+F 2 "MyLibs:PCS.06.A" H 9050 1200 50  0001 C CNN
+F 3 "~" H 9050 1200 50  0001 C CNN
+	1    9150 1150
+	-1   0    0    -1
+$EndComp
+Text Notes 950  3500 0    50   ~ 0
+ASR00012
+$Comp
+L power:GND #PWR0107
+U 1 1 61076EBD
+P 1550 3400
+F 0 "#PWR0107" H 1550 3150 50  0001 C CNN
+F 1 "GND" H 1555 3227 50  0000 C CNN
+F 2 "" H 1550 3400 50  0001 C CNN
+F 3 "" H 1550 3400 50  0001 C CNN
+	1    1550 3400
+	1    0    0    -1
+$EndComp
+$Comp
+L power:VBUS #PWR0108
+U 1 1 61076EC3
+P 1550 3050
+F 0 "#PWR0108" H 1550 2900 50  0001 C CNN
+F 1 "VBUS" H 1565 3223 50  0000 C CNN
+F 2 "" H 1550 3050 50  0001 C CNN
+F 3 "" H 1550 3050 50  0001 C CNN
+	1    1550 3050
+	1    0    0    -1
+$EndComp
+Wire Wire Line
+	1300 3200 1550 3200
+Wire Wire Line
+	1550 3200 1550 3050
+Wire Wire Line
+	1550 3400 1550 3300
+Wire Wire Line
+	1300 3300 1550 3300
+$Comp
+L Connector_Generic:Conn_01x02 J1
+U 1 1 61076ECD
+P 1100 3200
+F 0 "J1" H 1018 3417 50  0000 C CNN
+F 1 " micro JST SH" H 1018 3326 50  0000 C CNN
+F 2 "MyLibs:S2B-ZR-SM4A-TFLFSN" H 1100 3200 50  0001 C CNN
+F 3 "~" H 1100 3200 50  0001 C CNN
+	1    1100 3200
+	-1   0    0    -1
+$EndComp
+Text Notes 3200 1000 0    50   ~ 0
+1A
+$Comp
+L power:+1V8 #PWR0109
+U 1 1 61395600
+P 11450 2500
+F 0 "#PWR0109" H 11450 2350 50  0001 C CNN
+F 1 "+1V8" H 11465 2673 50  0000 C CNN
+F 2 "" H 11450 2500 50  0001 C CNN
+F 3 "" H 11450 2500 50  0001 C CNN
+	1    11450 2500
+	1    0    0    -1
+$EndComp
+$Comp
+L power:GND #PWR?
+U 1 1 6146F04B
+P 9700 1000
+F 0 "#PWR?" H 9700 750 50  0001 C CNN
+F 1 "GND" H 9705 827 50  0000 C CNN
+F 2 "" H 9700 1000 50  0001 C CNN
+F 3 "" H 9700 1000 50  0001 C CNN
+	1    9700 1000
+	1    0    0    -1
+$EndComp
+Wire Wire Line
+	9400 1100 9400 1200
+Wire Wire Line
+	9400 1100 9400 1000
+Connection ~ 9400 1100
+Wire Wire Line
+	9400 1000 9700 1000
+Connection ~ 9400 1000
 $EndSCHEMATC

Commit message: Final review
Parts:
- removed AE1: ACAG0301-1575-T, MyLibs:ACAG0301-1575-T, symbol Device:Antenna_Chip
- added U10: ACAG-0301-1575-T, MyLibs:ACAG0301-1575-T, symbol myPartsLibrary:ACAG-0301-1575-T
- C12: value 3.5pF -> 6.8pF
- L3: value 22nH -> 6.8nH
Connections:
- net GND: now also U10.2 (Pin_2), U10.3 (Pin_3); no longer J6.1 (Pin_1), J6.2 (Pin_2)
- net at L1.2: now also U10.1 (Pin_1)
- no-connect marks 80 -> 82
Changed lines of the file:
@@
 P 9650 1550
 F 0 "L3" V 9604 1628 50  0000 L CNN
-F 1 "22nH" V 9695 1628 50  0000 L CNN
+F 1 "6.8nH" V 9695 1628 50  0000 L CNN
 F 2 "Inductor_SMD:L_0402_1005Metric" H 9650 1550 50  0001 C CNN
 F 3 "~" H 9650 1550 50  0001 C CNN
@@
 P 10000 1300
 F 0 "C12" V 9850 1250 50  0000 L CNN
-F 1 "3.5pF" V 10150 1200 50  0000 L CNN
+F 1 "6.8pF" V 10150 1200 50  0000 L CNN
 F 2 "Capacitor_SMD:C_0402_1005Metric" H 10038 1150 50  0001 C CNN
 F 3 "~" H 10000 1300 50  0001 C CNN
@@
 $EndComp
 $Comp
-L Device:Antenna_Chip AE1
-U 1 1 5E770DC6
-P 5800 3200
-F 0 "AE1" H 5656 3327 50  0000 R CNN
-F 1 "ACAG0301-1575-T" H 5656 3236 50  0000 R CNN
-F 2 "MyLibs:ACAG0301-1575-T" H 5700 3375 50  0001 C CNN
-F 3 "~" H 5700 3375 50  0001 C CNN
-	1    5800 3200
-	-1   0    0    -1
-$EndComp
-$Comp
 L power:GND #PWR030
 U 1 1 5E772CDE
-P 5700 3450
-F 0 "#PWR030" H 5700 3200 50  0001 C CNN
-F 1 "GND" H 5705 3277 50  0000 C CNN
-F 2 "" H 5700 3450 50  0001 C CNN
-F 3 "" H 5700 3450 50  0001 C CNN
-	1    5700 3450
-	1    0    0    -1
-$EndComp
-Wire Wire Line
-	5700 3450 5700 3300
+P 6000 3600
+F 0 "#PWR030" H 6000 3350 50  0001 C CNN
+F 1 "GND" H 6005 3427 50  0000 C CNN
+F 2 "" H 6000 3600 50  0001 C CNN
+F 3 "" H 6000 3600 50  0001 C CNN
+	1    6000 3600
+	1    0    0    -1
+$EndComp
 $Comp
 L pspice:INDUCTOR L1
@@
 	1    0    0    -1
 $EndComp
-$Comp
-L power:GND #PWR?
-U 1 1 6146F04B
-P 9700 1000
-F 0 "#PWR?" H 9700 750 50  0001 C CNN
-F 1 "GND" H 9705 827 50  0000 C CNN
-F 2 "" H 9700 1000 50  0001 C CNN
-F 3 "" H 9700 1000 50  0001 C CNN
-	1    9700 1000
-	1    0    0    -1
-$EndComp
-Wire Wire Line
-	9400 1100 9400 1200
-Wire Wire Line
-	9400 1100 9400 1000
-Connection ~ 9400 1100
-Wire Wire Line
-	9400 1000 9700 1000
-Connection ~ 9400 1000
+Wire Wire Line
+	9400 1200 9500 1200
+Wire Wire Line
+	9500 1200 9500 1800
+Wire Wire Line
+	9500 1800 9650 1800
+Connection ~ 9650 1800
+NoConn ~ 9400 1000
+NoConn ~ 9400 1100
+$Comp
+L myPartsLibrary:ACAG-0301-1575-T U10
+U 1 1 619982B3
+P 5700 3550
+F 0 "U10" H 5658 4065 50  0000 C CNN
+F 1 "ACAG-0301-1575-T" H 5658 3974 50  0000 C CNN
+F 2 "MyLibs:ACAG0301-1575-T" H 5700 3550 50  0001 C CNN
+F 3 "" H 5700 3550 50  0001 C CNN
+	1    5700 3550
+	1    0    0    -1
+$EndComp
+Wire Wire Line
+	5900 3400 6000 3400
+Wire Wire Line
+	6000 3400 6000 3500
+Wire Wire Line
+	5900 3500 6000 3500
+Connection ~ 6000 3500
+Wire Wire Line
+	6000 3500 6000 3600
 $EndSCHEMATC

Commit message: Fixed capacitor footprints
Parts:
- C3, C4: footprint Capacitor_SMD:C_0402_1005Metric -> Capacitor_SMD:C_0805_2012Metric
Changed lines of the file:
@@
 F 0 "C4" H 2415 5896 50  0000 L CNN
 F 1 "100uF" H 2415 5805 50  0000 L CNN
-F 2 "Capacitor_SMD:C_0402_1005Metric" H 2338 5700 50  0001 C CNN
+F 2 "Capacitor_SMD:C_0805_2012Metric" H 2338 5700 50  0001 C CNN
 F 3 "~" H 2300 5850 50  0001 C CNN
 	1    2300 5850
@@
 F 0 "C3" H 2315 7696 50  0000 L CNN
 F 1 "100uF" H 2315 7605 50  0000 L CNN
-F 2 "Capacitor_SMD:C_0402_1005Metric" H 2238 7500 50  0001 C CNN
+F 2 "Capacitor_SMD:C_0805_2012Metric" H 2238 7500 50  0001 C CNN
 F 3 "~" H 2200 7650 50  0001 C CNN
 	1    2200 7650
